File: PiZeroAudio.sch (EAGLE design)
At the start: 9 parts

Commit message: Added Board
Parts:
- added J1: 1X2-3.5MM, adafruit:1X2-3.5MM
- C1, C2: value (none) -> 33nF; device eagle-ltspice:C -> adafruit:C-USC0805
- C3, C4: value (none) -> 47uF
- R1, R3: value (none) -> 270
- R2, R4: value (none) -> 150
Connections:
- new net +5V: J1.2, U$1.5V0@1, U$1.5V0@2
- new net GND: C1.2, C2.2, J1.1, R2.1, R4.1, U$1.GND@1, U$1.GND@2, U$1.GND@3, U$1.GND@4, U$1.GND@5, U$1.GND@6, U$1.GND@7, U$1.GND@8
- new net N$1: C1.1, C3.+, R1.1, R2.2
- new net N$3: C2.1, C4.+, R3.1, R4.2
- new net PWM-LEFT: R1.2, U$1.GPIO18
- new net PWM-RIGHT: R3.2, U$1.GPIO13
Other:
- moved on the sheet: C1, C2, C3, C4, R1, R2, R3, R4, U$1
Changed lines of the file:
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@@
 <parts>
 <part name="U$1" library="RPI-Zero" deviceset="RPI-ZERO" device=""/>
-<part name="C1" library="eagle-ltspice" library_urn="urn:adsk.eagle:library:217" deviceset="C" device="" package3d_urn="urn:adsk.eagle:package:13265/1"/>
-<part name="C2" library="eagle-ltspice" library_urn="urn:adsk.eagle:library:217" deviceset="C" device="" package3d_urn="urn:adsk.eagle:package:13265/1"/>
-<part name="C3" library="adafruit" deviceset="CPOL-US" device="085CS-1AR"/>
-<part name="C4" library="adafruit" deviceset="CPOL-US" device="085CS-1AR"/>
-<part name="R1" library="adafruit" deviceset="R-US_" device="R0805"/>
-<part name="R2" library="adafruit" deviceset="R-US_" device="R0805"/>
-<part name="R3" library="adafruit" deviceset="R-US_" device="R0805"/>
-<part name="R4" library="adafruit" deviceset="R-US_" device="R0805"/>
+<part name="C1" library="adafruit" deviceset="C-US" device="C0805" value="33nF"/>
+<part name="C2" library="adafruit" deviceset="C-US" device="C0805" value="33nF"/>
+<part name="C3" library="adafruit" deviceset="CPOL-US" device="085CS-1AR" value="47uF"/>
+<part name="C4" library="adafruit" deviceset="CPOL-US" device="085CS-1AR" value="47uF"/>
+<part name="R1" library="adafruit" deviceset="R-US_" device="R0805" value="270"/>
+<part name="R2" library="adafruit" deviceset="R-US_" device="R0805" value="150"/>
+<part name="R3" library="adafruit" deviceset="R-US_" device="R0805" value="270"/>
+<part name="R4" library="adafruit" deviceset="R-US_" device="R0805" value="150"/>
+<part name="SUPPLY1" library="supply2" library_urn="urn:adsk.eagle:library:372" deviceset="GND" device=""/>
+<part name="SUPPLY2" library="supply2" library_urn="urn:adsk.eagle:library:372" deviceset="GND" device=""/>
+<part name="5V0@1" library="supply1" library_urn="urn:adsk.eagle:library:371" deviceset="+5V" device=""/>
+<part name="J1" library="adafruit" deviceset="1X2" device="-3.5MM"/>
+<part name="P+2" library="supply1" library_urn="urn:adsk.eagle:library:371" deviceset="+5V" device=""/>
+<part name="SUPPLY3" library="supply2" library_urn="urn:adsk.eagle:library:372" deviceset="GND" device=""/>
 </parts>
 <sheets>
@@
 </plain>
 <instances>
-<instance part="U$1" gate="G$1" x="48.26" y="55.88"/>
-<instance part="C1" gate="G$1" x="106.68" y="93.98"/>
-<instance part="C2" gate="G$1" x="109.22" y="66.04"/>
-<instance part="C3" gate="G$1" x="127" y="93.98"/>
-<instance part="C4" gate="G$1" x="127" y="76.2"/>
-<instance part="R1" gate="G$1" x="96.52" y="45.72"/>
-<instance part="R2" gate="G$1" x="114.3" y="45.72"/>
-<instance part="R3" gate="G$1" x="134.62" y="45.72"/>
-<instance part="R4" gate="G$1" x="147.32" y="45.72"/>
+<instance part="U$1" gate="G$1" x="50.8" y="81.28"/>
+<instance part="C1" gate="G$1" x="99.06" y="83.82"/>
+<instance part="C2" gate="G$1" x="99.06" y="43.18"/>
+<instance part="C3" gate="G$1" x="109.22" y="88.9" rot="R90"/>
+<instance part="C4" gate="G$1" x="111.76" y="48.26" rot="R90"/>
+<instance part="R1" gate="G$1" x="91.44" y="99.06" rot="R90"/>
+<instance part="R2" gate="G$1" x="91.44" y="83.82" rot="R90"/>
+<instance part="R3" gate="G$1" x="91.44" y="55.88" rot="R90"/>
+<instance part="R4" gate="G$1" x="91.44" y="43.18" rot="R90"/>
+<instance part="SUPPLY1" gate="GND" x="91.44" y="35.56"/>
+<instance part="SUPPLY2" gate="GND" x="91.44" y="76.2"/>
+<instance part="5V0@1" gate="1" x="86.36" y="111.76"/>
+<instance part="J1" gate="G$1" x="139.7" y="106.68" rot="R180"/>
+<instance part="P+2" gate="1" x="147.32" y="111.76"/>
+<instance part="SUPPLY3" gate="GND" x="147.32" y="101.6"/>
 </instances>
 <busses>
 </busses>
 <nets>
+<net name="N$1" class="0">
+<segment>
+<pinref part="R1" gate="G$1" pin="1"/>
+<pinref part="R2" gate="G$1" pin="2"/>
+<wire x1="91.44" y1="93.98" x2="91.44" y2="88.9" width="0.1524" layer="91"/>
+<wire x1="91.44" y1="88.9" x2="99.06" y2="88.9" width="0.1524" layer="91"/>
+<junction x="91.44" y="88.9"/>
+<pinref part="C1" gate="G$1" pin="1"/>
+<wire x1="99.06" y1="88.9" x2="99.06" y2="86.36" width="0.1524" layer="91"/>
+<pinref part="C3" gate="G$1" pin="+"/>
+<wire x1="99.06" y1="88.9" x2="106.68" y2="88.9" width="0.1524" layer="91"/>
+<junction x="99.06" y="88.9"/>
+</segment>
+</net>
+<net name="N$3" class="0">
+<segment>
+<pinref part="R3" gate="G$1" pin="1"/>
+<pinref part="R4" gate="G$1" pin="2"/>
+<wire x1="91.44" y1="50.8" x2="91.44" y2="48.26" width="0.1524" layer="91"/>
+<wire x1="91.44" y1="48.26" x2="99.06" y2="48.26" width="0.1524" layer="91"/>
+<junction x="91.44" y="48.26"/>
+<pinref part="C2" gate="G$1" pin="1"/>
+<wire x1="99.06" y1="48.26" x2="99.06" y2="45.72" width="0.1524" layer="91"/>
+<pinref part="C4" gate="G$1" pin="+"/>
+<wire x1="99.06" y1="48.26" x2="109.22" y2="48.26" width="0.1524" layer="91"/>
+<junction x="99.06" y="48.26"/>
+</segment>
+</net>
+<net name="GND" class="0">
+<segment>
+<pinref part="C2" gate="G$1" pin="2"/>
+<pinref part="R4" gate="G$1" pin="1"/>
+<wire x1="99.06" y1="38.1" x2="91.44" y2="38.1" width="0.1524" layer="91"/>
+<pinref part="SUPPLY1" gate="GND" pin="GND"/>
+<junction x="91.44" y="38.1"/>
+</segment>
+<segment>
+<pinref part="C1" gate="G$1" pin="2"/>
+<pinref part="R2" gate="G$1" pin="1"/>
+<wire x1="99.06" y1="78.74" x2="91.44" y2="78.74" width="0.1524" layer="91"/>
+<pinref part="SUPPLY2" gate="GND" pin="GND"/>
+<junction x="91.44" y="78.74"/>
+</segment>
+<segment>
+<pinref part="SUPPLY3" gate="GND" pin="GND"/>
+<pinref part="J1" gate="G$1" pin="1"/>
+<wire x1="147.32" y1="104.14" x2="144.78" y2="104.14" width="0.1524" layer="91"/>
+</segment>
+<segment>
+<pinref part="U$1" gate="G$1" pin="GND@8"/>
+<wire x1="76.2" y1="106.68" x2="78.74" y2="106.68" width="0.1524" layer="91"/>
+</segment>
+<segment>
+<pinref part="U$1" gate="G$1" pin="GND@4"/>
+<wire x1="76.2" y1="96.52" x2="78.74" y2="96.52" width="0.1524" layer="91"/>
+</segment>
+<segment>
+<pinref part="U$1" gate="G$1" pin="GND@5"/>
+<wire x1="76.2" y1="88.9" x2="78.74" y2="88.9" width="0.1524" layer="91"/>
+</segment>
+<segment>
+<pinref part="U$1" gate="G$1" pin="GND@6"/>
+<wire x1="76.2" y1="76.2" x2="78.74" y2="76.2" width="0.1524" layer="91"/>
+</segment>
+<segment>
+<pinref part="U$1" gate="G$1" pin="GND@7"/>
+<wire x1="76.2" y1="71.12" x2="78.74" y2="71.12" width="0.1524" layer="91"/>
+</segment>
+<segment>
+<pinref part="U$1" gate="G$1" pin="GND@3"/>
+<wire x1="27.94" y1="63.5" x2="25.4" y2="63.5" width="0.1524" layer="91"/>
+</segment>
+<segment>
+<pinref part="U$1" gate="G$1" pin="GND@2"/>
+<wire x1="27.94" y1="81.28" x2="25.4" y2="81.28" width="0.1524" layer="91"/>
+</segment>
+<segment>
+<pinref part="U$1" gate="G$1" pin="GND@1"/>
+<wire x1="27.94" y1="101.6" x2="25.4" y2="101.6" width="0.1524" layer="91"/>
+</segment>
+</net>
+<net name="PWM-LEFT" class="0">
+<segment>
+<pinref part="R1" gate="G$1" pin="2"/>
+<wire x1="91.44" y1="104.14" x2="99.06" y2="104.14" width="0.1524" layer="91"/>
+<label x="99.06" y="104.14" size="1.778" layer="95" xref="yes"/>
+<pinref part="U$1" gate="G$1" pin="GPIO18"/>
+<wire x1="76.2" y1="99.06" x2="86.36" y2="99.06" width="0.1524" layer="91"/>
+<wire x1="86.36" y1="99.06" x2="86.36" y2="104.14" width="0.1524" layer="91"/>
+<wire x1="86.36" y1="104.14" x2="91.44" y2="104.14" width="0.1524" layer="91"/>
+<junction x="91.44" y="104.14"/>
+</segment>
+</net>
+<net name="PWM-RIGHT" class="0">
+<segment>
+<pinref part="R3" gate="G$1" pin="2"/>
+<label x="101.6" y="60.96" size="1.778" layer="95" xref="yes"/>
+<wire x1="101.6" y1="60.96" x2="91.44" y2="60.96" width="0.1524" layer="91"/>
+</segment>
+<segment>
+<pinref part="U$1" gate="G$1" pin="GPIO13"/>
+<wire x1="27.94" y1="71.12" x2="22.86" y2="71.12" width="0.1524" layer="91"/>
+<wire x1="22.86" y1="71.12" x2="22.86" y2="48.26" width="0.1524" layer="91"/>
+<wire x1="22.86" y1="48.26" x2="30.48" y2="48.26" width="0.1524" layer="91"/>
+<label x="30.48" y="48.26" size="1.778" layer="95" xref="yes"/>
+</segment>
+</net>
+<net name="+5V" class="0">
+<segment>
+<pinref part="U$1" gate="G$1" pin="5V0@2"/>
+<pinref part="5V0@1" gate="1" pin="+5V"/>
+<wire x1="76.2" y1="109.22" x2="86.36" y2="109.22" width="0.1524" layer="91"/>
+<pinref part="U$1" gate="G$1" pin="5V0@1"/>
+<wire x1="76.2" y1="111.76" x2="76.2" y2="109.22" width="0.1524" layer="91"/>
+<junction x="76.2" y="109.22"/>
+<label x="86.36" y="109.22" size="1.778" layer="95" xref="yes"/>
+</segment>
+<segment>
+<pinref part="J1" gate="G$1" pin="2"/>
+<wire x1="144.78" y1="106.68" x2="147.32" y2="106.68" width="0.1524" layer="91"/>
+<pinref part="P+2" gate="1" pin="+5V"/>
+<wire x1="147.32" y1="106.68" x2="147.32" y2="109.22" width="0.1524" layer="91"/>
+<label x="147.32" y="106.68" size="1.778" layer="95" xref="yes"/>
+</segment>
+</net>
 </nets>
 </sheet>
@@
 will not be understood (or retained) with this version.
 </note>
-<note version="8.3" severity="warning">
-Since Version 8.3, EAGLE supports the association of 3D packages
-with devices in libraries, schematics, and board files. Those 3D
-packages will not be understood (or retained) with this version.
-</note>
 </compatibility>
