File: PiZeroAudio.sch (EAGLE design)
At the start: 60 parts, among them CN1 1X4-BIG, CON1 RPI-ZERO, J1 1X2-3.5MM, U1 TXB0104PWR, U2 LSM6DS33, U3 NC7WZ16, U4 TPA3144D2PWPR

Commit message: Pre- grove connector
Parts:
- removed CN1: 1X4-BIG, adafruit:1X4-BIG
- removed D1: (no value), diode:SCHOTTKY-DIODESMD
- added J2: 4X1-LOCKING, HappyBrackets:4X1-LOCKING
- added Q1: DMG2305UX, HappyBrackets:DMG2305UX
- added R18: 33K, adafruit:R-US_R0603
- added R19: 10R, adafruit:R-US_R0603
- added U5: TPA3144D2PWPR, HappyBrackets:TPA3144D2PWPR
- J1: value 1X2-3.5MM -> 2X1-LOCKING; device adafruit:1X2-3.5MM -> HappyBrackets:2X1-LOCKING
- JP1: value GPIO -> (none); device adafruit:PINHD-2X4 -> adafruit:PINHD-1X3
- JP2: value (none) -> GPIO; device adafruit:PINHD-1X3 -> adafruit:PINHD-2X4
- R1, R2: value 10K -> 220
- R10: value 39K -> 1K8
- R11: value 56K -> 10K
- R12: value 33K -> 47K
- R13: value 33K -> 10K
- R14: value 33K -> 39K
- R15: value 10R -> 56K
- R16, R17: value 220 -> 33K
- R3: value 220 -> 10K
- R4: value 100 -> 10K
- R5, R8: value 1K8 -> 220
- R6: value 220 -> 100
- R7: value 100 -> 1K8
- R9: value 10K -> 100
- U4: value TPA3144D2PWPR -> DMMT5401; device HappyBrackets:TPA3144D2PWPR -> HappyBrackets:DMMT5401
Connections:
- removed net PWR-IN: D1.A, J1.2
- new net +5V-IN: J1.1, Q1.S, U4G$1.E
- new net N$22: R13.1, U4G$1.B, U4G$2.B, U4G$2.C
- new net N$27: Q1.G, R12.1, U4G$1.C
- net +3V3: now also JP1.1, R1.2, R3.1, R4.1; no longer JP2.1, R1.1, R17.2, R2.1
- net +5V: now also Q1.D, R19.2, U4G$2.E, U5.15-PVCC, U5.16-PVCC, U5.27-PVCC, U5.28-PVCC; no longer D1.C, R15.2, U4.15-PVCC, U4.16-PVCC, U4.27-PVCC, U4.28-PVCC
- net /MUTE: now also R11.1; no longer R9.1
- net AGND: now also J1.2, R10.1, R13.2, R14.2, R16.2, R6.1, R9.1, U5.19-GND, U5.1SPW-13, U5.24-GND, U5.GND-10, U5.GND-PAD; no longer J1.1, R10.2, R4.1, R5.1, R8.1, U4.19-GND, U4.1SPW-13, U4.24-GND, U4.GND-10, U4.GND-PAD
- net AUDIO-LEFT: now also R7.2, U5.LINP-3; no longer R5.2, U4.LINP-3
- net AUDIO-RIGHT: now also R10.2, U5.RINP-12; no longer R8.2, U4.RINP-12
- net GND: now also JP1.3, JP2.2, JP2.4, JP2.6, JP2.8, R2.1; no longer JP1.2, JP1.4, JP1.6, JP1.8, JP2.3, R16.1
- net L+: now also J2.4; no longer CN1.1
- net L-: now also J2.3; no longer CN1.2
- net N$1: now also R5.1, R6.2; no longer R3.1, R4.2
- net N$10: now also U5.17-BSPR; no longer U4.17-BSPR
- net N$11: now also JP2.1; no longer JP1.1
- net N$12: now also JP2.3; no longer JP1.3
- net N$13: now also U5.21-BSNR; no longer U4.21-BSNR
- net N$14: now also JP2.5; no longer JP1.5
- net N$15: now also JP2.7; no longer JP1.7
- net N$16: now also U5.22-BSNL; no longer U4.22-BSNL
- net N$17: now also U5.26-BSPL; no longer U4.26-BSPL
- net N$18: now also U5.25-OUTPL; no longer U4.25-OUTPL
- net N$19: now also U5.23-OUTNL; no longer U4.23-OUTNL
- net N$2: now also R5.2; no longer R3.2
- net N$20: now also U5.20-OUTNR; no longer U4.20-OUTNR
- net N$21: now also U5.18-OUTPR; no longer U4.18-OUTPR
- net N$23: now also R16.1, R17.2, U5.GAIN-6; no longer R12.1, R13.2, U4.GAIN-6
- net N$24: now also R17.1, R18.2, U5.SSCTRL-7; no longer R13.1, R14.2, U4.SSCTRL-7
- net N$25: now also R14.1, R15.2, U5.LIMTHRES-8; no longer R10.1, R11.2, U4.LIMTHRES-8
- net N$26: now also R15.1, R18.1, U5.GVDD-9, U5.LIMRATE-5; no longer R11.1, R14.1, U4.GVDD-9, U4.LIMRATE-5
- net N$3: now also R8.2; no longer R6.2
- net N$4: now also R8.1, R9.2; no longer R6.1, R7.2
- net N$5: now also R11.2, U5./FAULT-2, U5./SD-1; no longer R9.2, U4./FAULT-2, U4./SD-1
- net N$6: now also R2.2; no longer R16.2
- net N$7: now also U5.LINN-4; no longer U4.LINN-4
- net N$8: now also U5.RINN-11; no longer U4.RINN-11
- net N$9: now also R19.1, U5.AVCC-14; no longer R15.1, U4.AVCC-14
- net PWR-LED: now also JP1.2, R1.1; no longer JP2.2, R17.1
- net R+: now also J2.1; no longer CN1.4
- net R-: now also J2.2; no longer CN1.3
- net SCL: now also R4.2; no longer R2.2
- net SDA: now also R3.2; no longer R1.2
Other:
- moved on the sheet: R1, R10, R11, R12, R13, R14, R15, R16, R17, R2, R3, R4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
