File: PiZeroAudioI2SPam8403.sch (EAGLE design)
At the start: 60 parts, among them CON1 RPI-Header, J1 GROVE, J2 2X2HEADER, J3 JST, J4 AMP FCI 10103594-0001LF, J5 2X1-LOCKING, J6 GROVE, J7 4X1-LOCKING, Q1 DMG2305UX, U1 TXB0104PWR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

Commit message: Swapped position of Mosfet Capacitively coupled Audio Set OE of I2C translator to GND Set Mute so it floats to +5
Parts:
- removed U5: DMMT5401, HappyBrackets:DMMT5401
- added C23, C24: 1uF, rcl:C-EUC0603
- added R16, R17: 160K, adafruit:R-US_R0603
- added R18: 1K, adafruit:R-US_R0603
- C1, C10, C12, C15, C2, C21, C3, C6: MF (none) -> MULTICOMP; MPN (none) -> MC0603F104Z500CT; OC_FARNELL (none) -> 1759123
- C11, C14, C16, C4: MF (none) -> AVX; MPN (none) -> F931C106MAA; OC_FARNELL (none) -> 2852673
- C13, C17, C18, C19, C5, C7, CON1, D1, J1, J2, J5, J6, J7, JP1, LED1, R8, SH1, SH2, U6, U7, U8: OC_FARNELL (none) -> unknown
- C20: MF (none) -> VISHAY; MPN (none) -> 293D477X9010E2TE3; OC_FARNELL (none) -> 2353079
- C22: MF (none) -> MURATA; MPN (none) -> GRM188R61A226ME15D; OC_FARNELL (none) -> 2426957
- C8, C9: MF (none) -> TAIYO YUDEN; MPN (none) -> TMK107ABJ225KA-T; OC_FARNELL (none) -> 2503459
- J3: MF (none) -> JST (JAPAN SOLDERLESS TERMINALS); MPN (none) -> S2B-PH-SM4-TB(LF)(SN); OC_FARNELL (none) -> 9492615
- J4: MF (none) -> AMPHENOL ICC (FCI); MPN (none) -> 10103594-0001LF; OC_FARNELL (none) -> 2293752
- L1: value IFSC1515AHER2R2M01 -> 2.2uH; MF (none) -> VISHAY; MPN (none) -> IFSC1515AHER2R2M01; OC_FARNELL (none) -> 2352690
- Q1: MF (none) -> DIODES INC.; MPN (none) -> DMG2305UX-7; OC_FARNELL (none) -> 2543533
- R1, R2: MF (none) -> YAGEO; MPN (none) -> RC0603FR-07220RL; OC_FARNELL (none) -> 2421863
- R10: value 10K -> 180; MF (none) -> PANASONIC ELECTRONIC COMPONENTS; MPN (none) -> ERJ3EKF4700V; OC_FARNELL (none) -> 2303120
- R11, R3, R4: MF (none) -> YAGEO; MPN (none) -> RC0603FR-0710KL; OC_FARNELL (none) -> 2133286
- R12, R13: MF (none) -> VISHAY; MPN (none) -> CRCW0603750KFKEA; OC_FARNELL (none) -> 1152123
- R14, R15: MF (none) -> PANASONIC ELECTRONIC COMPONENTS; MPN (none) -> ERJ-3EKF1003V; OC_FARNELL (none) -> 2289601
- R5, R6: MF (none) -> PANASONIC ELECTRONIC COMPONENTS; MPN (none) -> ERJ3EKF4700V; OC_FARNELL (none) -> 2303120
- R7: MF (none) -> VISHAY; MPN (none) -> CRCW06031K00FKEA; OC_FARNELL (none) -> 1469740
- R9: value 47K -> 180; MF (none) -> PANASONIC ELECTRONIC COMPONENTS; MPN (none) -> ERJ3EKF4700V; OC_FARNELL (none) -> 2303120
- U1: MF (none) -> TEXAS INSTRUMENTS; MPN (none) -> TXB0104PWR; OC_FARNELL (none) -> 1607891
- U2: MF (none) -> STMICROELECTRONICS; MPN (none) -> LSM6DS33TR; OC_FARNELL (none) -> 2762756
- U3: MF (none) -> TEXAS INSTRUMENTS; MPN (none) -> PCM5101AQPWRQ1; OC_FARNELL (none) -> 2402250
- U4: MF (none) -> MICROCHIP; MPN (none) -> MCP73831T-2ACI/OT; OC_FARNELL (none) -> 1332158
Connections:
- removed net N$22: R10.1, U5G$1.B, U5G$2.B, U5G$2.C
- removed net N$27: Q1.G, R9.1, U5G$1.C
- new net N$10: R17.2, U7.10-INR
- new net N$13: C23.1, R16.1
- new net N$8: R16.2, U7.7-INL
- new net OE: CON1.GPIO20, U1.OE
- net +3V3: no longer U1.OE, U6.OE
- net +5V: now also C18.1, C19.1, C20.+, R11.1, U7.PVDD-13, U7.PVDD-4
- net +5V-IN: now also Q1.D; no longer Q1.S, U5G$1.E
- net +5VCHARGE: now also Q1.S; no longer Q1.D, U5G$2.E
- net /MUTE: now also R11.2, R18.1, R18.2, U7.12-/SHND, U7.5-/MUTE; no longer R11.1
- net AGND: now also Q1.G; no longer R10.2, R9.2
- net AN3V3: no longer C18.1, C19.1, C20.+, U7.PVDD-13, U7.PVDD-4
- net AUDIO-LEFT: now also C23.2, R9.1; no longer U7.7-INL
- net AUDIO-RIGHT: now also R10.1; no longer U7.10-INR
- net GND: now also C24.2, R10.2, R9.2, U6.OE
- net N$5: now also C24.1, R17.1; no longer R11.2, U7.12-/SHND, U7.5-/MUTE
Other:
- note removed: "Switch bypass"
- moved on the sheet: R10, R9
