File: Pi-Breakout.brd (EAGLE design)
At the start: 100 x 100 mm, 43 parts, among them CON1 RPI-ZERO, CON2 RPI-ZERO, J1 2X1-LOCKING, J2 2X1-LOCKING, U1 TC1014-3.3V, U2 TC1014-3.3V

Commit message: Added Second CIRCUIT
Parts:
- removed 3V3-OUT1: (no value), adafruit:1X03
- removed DIG_V: 2X2HEADER, HappyBrackets:2X2
- added J3: 1X2EDGE, HappyBrackets:1X2_EDGE
- added U$1: 1X3EDGE, HappyBrackets:1X3_EDGE
- J2: value 2X1-LOCKING -> 1X2EDGE; device HappyBrackets:22-23-2021 -> HappyBrackets:1X2_EDGE
- moved 5V1 86.0 mm to (78.9, 94.8)
- moved 5V2 86.0 mm to (84.6, 94.8)
- moved GND1 86.0 mm to (91.2, 94.7)
- moved GND2 86.0 mm to (96.8, 94.7)
- moved J1 86.0 mm to (69.4, 88.6)
- moved L1 86.0 mm to (75.0, 88.4)
- moved L2 86.0 mm to (77.8, 88.4)
- moved L3 86.0 mm to (80.8, 88.5)
- moved L4 86.0 mm to (83.5, 88.6)
- moved L5 86.0 mm to (87.3, 88.3)
- moved L6 86.0 mm to (89.9, 88.4)
- moved L7 86.0 mm to (92.9, 88.4)
- moved L8 86.0 mm to (95.7, 88.3)
- moved 3V3-OUT 51.5 mm to (79.8, 77.6)
- moved C1 51.5 mm to (82.3, 70.4)
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Connections:
- net 0_IN: now also J2.P$2; no longer J2.2
- net 5_IN: now also J2.P$1; no longer J2.1
- net ANA_GND: now also U$1.P$2; no longer 3V3-OUT1.2
- net AN_5V: now also U$1.P$3; no longer 3V3-OUT1.1
- net DIG_5V: now also J3.P$1; no longer DIG_V.3, DIG_V.4
- net DIG_GND: now also J3.P$2; no longer DIG_V.1, DIG_V.2
- net N$42: now also U$1.P$1; no longer 3V3-OUT1.3
Routing:
- net GND_9_B: track 10.7 -> 45.7 mm
- net GND_20_B: track 13.7 -> 48.0 mm
- net 3V3_1_B: track 11.1 -> 44.8 mm
- net GND_39_B: track 11.0 -> 44.7 mm
- net GND_14_B: track 13.8 -> 47.2 mm
- net GND_25_B: track 11.1 -> 44.2 mm
- net GND_6_B: track 13.9 -> 47.0 mm
- net 5V1_B: track 13.7 -> 46.8 mm
- net 3V3_17_B: track 11.0 -> 43.6 mm
- net GND_30_B: track 13.7 -> 46.4 mm
- net GND@7: track 14.6 -> 47.0 mm
- net 5V0_B: track 14.1 -> 46.5 mm
- net GND_34_PI: track 16.3 -> 34.5 mm
- net 5V0_PI: track 15.7 -> 33.6 mm
- net GND_9_PI: track 13.3 -> 31.0 mm
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- added copper zone on layer 1, net ANA_GND
- added copper zone on layer 16, net ANA_GND
- added copper zone on layer 1, net AN_5V
- added copper zone on layer 1, net DIG_5V
- added copper zone on layer 1, net DIG_GND
- added copper zone on layer 16, net DIG_GND

Commit message: Added Breakout
Parts:
- L1, L2, L5, L6: value BLM31A -> 300
- L3, L7: value BLM31A -> 1K
- L4, L8: value BLM31A -> 1k
Changed lines of the file:
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@@
 <layer number="18" name="Vias" color="2" fill="1" visible="yes" active="yes"/>
 <layer number="19" name="Unrouted" color="6" fill="1" visible="yes" active="yes"/>
-<layer number="20" name="Dimension" color="24" fill="1" visible="yes" active="yes"/>
+<layer number="20" name="Dimension" color="24" fill="1" visible="no" active="yes"/>
 <layer number="21" name="tPlace" color="7" fill="1" visible="yes" active="yes"/>
 <layer number="22" name="bPlace" color="7" fill="1" visible="yes" active="yes"/>
@@
 <layer number="43" name="vRestrict" color="2" fill="10" visible="yes" active="yes"/>
 <layer number="44" name="Drills" color="7" fill="1" visible="no" active="yes"/>
-<layer number="45" name="Holes" color="7" fill="1" visible="no" active="yes"/>
+<layer number="45" name="Holes" color="7" fill="1" visible="yes" active="yes"/>
 <layer number="46" name="Milling" color="3" fill="1" visible="no" active="yes"/>
 <layer number="47" name="Measures" color="7" fill="1" visible="no" active="yes"/>
@@
 <text x="79.121" y="79.121" size="1.778" layer="25">0</text>
 <text x="81.3308" y="79.121" size="1.778" layer="25">3V3</text>
-<wire x1="0.2286" y1="49.5808" x2="99.9998" y2="49.5808" width="0.254" layer="25"/>
+<wire x1="-8.9154" y1="50.3428" x2="90.8558" y2="50.3428" width="0.254" layer="25"/>
 <text x="2.7178" y="39.7256" size="1.778" layer="25" rot="R90">+5</text>
 <text x="72.0598" y="60.5282" size="1.778" layer="25">Male</text>
@@
 <attribute name="VALUE" x="34.5694" y="50.9016" size="1.27" layer="27" rot="R90"/>
 </element>
-<element name="L1" library="HappyBrackets" library_urn="urn:adsk.eagle:library:5224691" package="SML1206" package3d_urn="urn:adsk.eagle:package:15829/1" value="BLM31A" x="74.9554" y="88.392" smashed="yes" rot="R90">
+<element name="L1" library="HappyBrackets" library_urn="urn:adsk.eagle:library:5224691" package="SML1206" package3d_urn="urn:adsk.eagle:package:15829/1" value="300" x="74.9554" y="88.392" smashed="yes" rot="R90">
 <attribute name="NAME" x="75.3016" y="83.5392" size="1.27" layer="25" rot="R90"/>
 </element>
-<element name="L2" library="HappyBrackets" library_urn="urn:adsk.eagle:library:5224691" package="SML1206" package3d_urn="urn:adsk.eagle:package:15829/1" value="BLM31A" x="77.8256" y="88.392" smashed="yes" rot="R90">
+<element name="L2" library="HappyBrackets" library_urn="urn:adsk.eagle:library:5224691" package="SML1206" package3d_urn="urn:adsk.eagle:package:15829/1" value="300" x="77.8256" y="88.392" smashed="yes" rot="R90">
 <attribute name="NAME" x="78.1972" y="83.336" size="1.27" layer="25" rot="R90"/>
 </element>
-<element name="L3" library="HappyBrackets" library_urn="urn:adsk.eagle:library:5224691" package="SML1206" package3d_urn="urn:adsk.eagle:package:15829/1" value="BLM31A" x="80.8228" y="88.519" smashed="yes" rot="R90">
+<element name="L3" library="HappyBrackets" library_urn="urn:adsk.eagle:library:5224691" package="SML1206" package3d_urn="urn:adsk.eagle:package:15829/1" value="1K" x="80.8228" y="88.519" smashed="yes" rot="R90">
 <attribute name="NAME" x="81.2198" y="83.5138" size="1.27" layer="25" rot="R90"/>
 </element>
-<element name="L4" library="HappyBrackets" library_urn="urn:adsk.eagle:library:5224691" package="SML1206" package3d_urn="urn:adsk.eagle:package:15829/1" value="BLM31A" x="83.4644" y="88.5698" smashed="yes" rot="R90">
+<element name="L4" library="HappyBrackets" library_urn="urn:adsk.eagle:library:5224691" package="SML1206" package3d_urn="urn:adsk.eagle:package:15829/1" value="1k" x="83.4644" y="88.5698" smashed="yes" rot="R90">
 <attribute name="NAME" x="84.0392" y="83.4122" size="1.27" layer="25" rot="R90"/>
 </element>
-<element name="L5" library="HappyBrackets" library_urn="urn:adsk.eagle:library:5224691" package="SML1206" package3d_urn="urn:adsk.eagle:package:15829/1" value="BLM31A" x="87.2998" y="88.2904" smashed="yes" rot="R90">
+<element name="L5" library="HappyBrackets" library_urn="urn:adsk.eagle:library:5224691" package="SML1206" package3d_urn="urn:adsk.eagle:package:15829/1" value="300" x="87.2998" y="88.2904" smashed="yes" rot="R90">
 <attribute name="NAME" x="88.027" y="83.336" size="1.27" layer="25" rot="R90"/>
 </element>
-<element name="L6" library="HappyBrackets" library_urn="urn:adsk.eagle:library:5224691" package="SML1206" package3d_urn="urn:adsk.eagle:package:15829/1" value="BLM31A" x="89.916" y="88.3666" smashed="yes" rot="R90">
+<element name="L6" library="HappyBrackets" library_urn="urn:adsk.eagle:library:5224691" package="SML1206" package3d_urn="urn:adsk.eagle:package:15829/1" value="300" x="89.916" y="88.3666" smashed="yes" rot="R90">
 <attribute name="NAME" x="90.5924" y="83.3614" size="1.27" layer="25" rot="R90"/>
 </element>
-<element name="L7" library="HappyBrackets" library_urn="urn:adsk.eagle:library:5224691" package="SML1206" package3d_urn="urn:adsk.eagle:package:15829/1" value="BLM31A" x="92.9386" y="88.3666" smashed="yes" rot="R90">
+<element name="L7" library="HappyBrackets" library_urn="urn:adsk.eagle:library:5224691" package="SML1206" package3d_urn="urn:adsk.eagle:package:15829/1" value="1K" x="92.9386" y="88.3666" smashed="yes" rot="R90">
 <attribute name="NAME" x="93.6404" y="83.3868" size="1.27" layer="25" rot="R90"/>
 </element>
-<element name="L8" library="HappyBrackets" library_urn="urn:adsk.eagle:library:5224691" package="SML1206" package3d_urn="urn:adsk.eagle:package:15829/1" value="BLM31A" x="95.7072" y="88.3158" smashed="yes" rot="R90">
+<element name="L8" library="HappyBrackets" library_urn="urn:adsk.eagle:library:5224691" package="SML1206" package3d_urn="urn:adsk.eagle:package:15829/1" value="1k" x="95.7072" y="88.3158" smashed="yes" rot="R90">
 <attribute name="NAME" x="96.282" y="83.209" size="1.27" layer="25" rot="R90"/>
 </element>
@@
 </polygon>
 <polygon width="0.508" layer="16">
-<vertex x="18.5928" y="49.53"/>
-<vertex x="17.8308" y="49.53"/>
+<vertex x="18.923" y="49.1998"/>
+<vertex x="17.8308" y="49.1998"/>
 <vertex x="17.8308" y="41.3258"/>
 <vertex x="29.9974" y="41.3004"/>
-<vertex x="29.8196" y="49.53"/>
+<vertex x="29.826734375" y="49.1998"/>
 </polygon>
 <via x="25.273" y="46.2534" extent="1-16" drill="0.35"/>
