File: PiZeroAudioI2S.sch (EAGLE design)
At the start: 69 parts, among them CON1 RPI-Header, J1 GROVE, J2 2X2HEADER, J3 2X1-LOCKING, J4 GROVE, J5 4X1-LOCKING, Q1 DMG2305UX, U1 TXB0104PWR, U2 LSM6DS33, U3 PCM5101A, U4 TXS0102, U5 TPA3144D2PWPR

Commit message: Added Breakout
Parts:
- R5, R6: MPN ERJ3EKF4700V -> RMCF0603FT76K8
Changed lines of the file:
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@@
 <part name="R5" library="adafruit" deviceset="R-US_" device="R0603" value="76K8">
 <attribute name="MF" value="PANASONIC ELECTRONIC COMPONENTS"/>
-<attribute name="MPN" value="ERJ3EKF4700V"/>
+<attribute name="MPN" value="RMCF0603FT76K8"/>
 <attribute name="OC_FARNELL" value="2303120"/>
 </part>
 <part name="R6" library="adafruit" deviceset="R-US_" device="R0603" value="76K8">
 <attribute name="MF" value="PANASONIC ELECTRONIC COMPONENTS"/>
-<attribute name="MPN" value="ERJ3EKF4700V"/>
+<attribute name="MPN" value="RMCF0603FT76K8"/>
 <attribute name="OC_FARNELL" value="2303120"/>
 </part>

Commit message: Update for Move account
Connections:
- net +5V: now also U4.OE
- net GND: now also C11.-; no longer C11.+, U4.OE
- net N$12: now also C11.+; no longer C11.-
Other:
- moved on the sheet: C11
