File: PiZeroHifi.brd (EAGLE design)
At the start: 100 x 80 mm, 45 parts, among them CON1 RPI-ZEROPI-ZERO-THRUHOLE, CON3 Audio Out, J1 GROVEGROVE-HORIZONTAL, J2 GROVEGROVE-HORIZONTAL, J3 GROVEGROVE-HORIZONTAL, U1 TXS0102, U2 LSM6DS33, U3 TC1014-3.3V, U4 PCM5101A, U5 PAM8403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

Commit message: Route HifiBoard
Parts:
- removed C1: 1500uF, HappyBrackets:CAP8MMX3.5MMX20MM
- removed R1: 10K, adafruit:R0603
- moved C20 114.6 mm to (62.7, 15.2), turned to 90 degrees
- moved C21 108.3 mm to (47.9, 12.9), turned to 90 degrees
- moved C19 106.6 mm to (62.7, 20.6), turned to 90 degrees
- moved C15 103.8 mm to (36.6, 20.3), turned to 90 degrees
- moved C8 103.6 mm to (54.3, 22.3)
- moved R10 103.3 mm to (44.4, 17.3), turned to 180 degrees
- moved C10 103.2 mm to (43.4, 12.3), turned to 270 degrees
- moved R11 102.8 mm to (44.4, 15.3), turned to 180 degrees
- moved R7 101.9 mm to (41.4, 20.4), turned to 90 degrees
- moved C12 96.4 mm to (44.7, 22.6)
- moved C18 95.6 mm to (60.3, 17.5), turned to 270 degrees
- moved C6 94.9 mm to (49.5, 17.7), turned to 180 degrees
- moved C22 94.1 mm to (50.3, 14.0), turned to 90 degrees
- moved U3 92.7 mm to (45.8, 19.8), turned to 270 degrees
- moved R9 92.5 mm to (37.8, 15.1), turned to 180 degrees
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Connections:
- removed net N$14: CON3.P$1, U5.1
- removed net N$15: CON3.P$2, U5.3
- removed net N$16: CON3.P$3, U5.14
- removed net N$17: CON3.P$4, U5.16
- removed net N$26: C23.2, R15.2, R16.1, U1.P$6
- new net +L: CON3.P$2, U5.1
- new net +R: CON3.P$3, U5.16
- new net -L: CON3.P$1, U5.3
- new net -R: CON3.P$4, U5.14
- net +5V: no longer C1.P$1
- net ACCEL_INT_1: now also CON1.13, U2.7; no longer CON1.11, U2.6
- net ACCEL_INT_2: now also CON1.11, U2.6; no longer CON1.13, U2.7
- net GND: no longer C1.P$2, R1.1
- net OE: now also C23.2, R15.2, R16.1, U1.P$6; no longer CON1.38, R1.2
Routing:
- net GND: track 0.00 -> 260.4 mm, vias 0 -> 14
- net +5V: track 0.00 -> 159.7 mm, vias 0 -> 2
- net +3V3: track 0.00 -> 135.0 mm, vias 0 -> 2
- net PCM_CLK: track 0.00 -> 59.4 mm, vias 0 -> 2
- net GPIO23: track 0.00 -> 50.9 mm, vias 0 -> 2
- net GPIO25: track 0.00 -> 44.2 mm, vias 0 -> 2
- net -R: track 0.00 -> 37.0 mm
- net +R: track 0.00 -> 35.9 mm
- net AN3V3: track 0.00 -> 32.8 mm, vias 0 -> 2
- net GPIO22: track 0.00 -> 30.6 mm
- net +L: track 0.00 -> 30.1 mm
- net /MUTE: track 0.00 -> 28.8 mm, vias 0 -> 1
- net GPIO21: track 0.00 -> 28.0 mm
- net OE: track 0.00 -> 26.6 mm, vias 0 -> 2
- net N$11: track 0.00 -> 26.4 mm
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- added copper zone on layer 1, net GND
- added copper zone on layer 16, net GND
Other:
- board size 100 x 80 mm -> 65.3 x 30.1 mm
